Commit message: Fix:update gopigo.xacro file

File: src/gopigo_description/urdf/gopigo.xacro (robot description, xacro)
@@ -1,6 +1,8 @@
 <?xml version='1.0'?>
-<robot name="gopigo" xmlns:xacro="http://www.ros.org/wiki/xacro">
+<robot name="gopigo3" xmlns:xacro="http://www.ros.org/wiki/xacro">
+  <!-- <link name='map'>
+  </link> -->
+ <!-- <link name='odom'/> -->
   <link name='base_link'>
-    <pose>0 0 0.1 0 0 0</pose>
     <inertial>
       <mass value="15.0"/>
@@ -93,4 +95,62 @@
     </inertial>
   </link>
+  <link name="gopigo3_body">
+    <visual>
+      <geometry>
+        <box size=".13 .1 .055"/>
+      </geometry>
+      <origin xyz="0 0 0" rpy=" 0 0 0"/>
+    </visual>
+    <collision name="collision">
+      <origin xyz="0 0 0" rpy="0 0 0"/>
+      <geometry>
+        <box size=".13 .1 .055"/>
+      </geometry>
+    </collision>
+    <inertial>
+      <origin xyz="0 0 0" rpy="0 0 0"/>
+      <mass value="5"/>
+      <inertia
+        ixx=".1" ixy="0.0" ixz="0.0"
+        iyy=".1" iyz="0.0"
+        izz=".1"/>
+    </inertial>
+  </link>
+ <!-- lidar
+  <link name="lidar">
+    <visual>
+      <geometry>
+        <cylinder radius="0.03" length="0.04"/>
+      </geometry>
+      <origin xyz="0 0 0" rpy=" 0 0 0"/>
+    </visual>
+    <collision name="collision">
+      <origin xyz="0 0 0" rpy=" 0 0 0"/>
+      <geometry>
+        <cylinder radius="0.03" length="0.04"/>
+      </geometry>
+    </collision>
+    <inertial>
+      <origin xyz="0 0 0" rpy=" 0 0 0"/>
+      <mass value="5"/>
+      <inertia
+        ixx=".1" ixy="0.0" ixz="0.0"
+        iyy=".1" iyz="0.0"
+        izz=".1"/>
+    </inertial>
+  </link>
+ -->
+  <!-- Joints -->
+  <!-- <joint type="floating" name="map_to_odom">
+    <parent link="map"/>
+    <child link="odom"/>
+    <origin xyz="0 0 0" rpy="0 0 0"/>
+  </joint>
+  <joint type="floating" name="odom_to_base">
+    <parent link="odom"/>
+    <child link="base_link"/>
+    <origin xyz="0 0 -0.036" rpy="0 0 0"/>
+  </joint>
+ -->
   <joint type="continuous" name="left_wheel_hinge">
     <origin xyz="0.03 0.05 0.036" rpy="0 0 0"/>
@@ -111,3 +171,15 @@
     <joint_properties damping="1.0" friction="1.0"/>
   </joint>
+  <joint type="fixed" name="base_to_body">
+    <origin xyz="0.015 0 0.0645" rpy=" 0 0 0"/>
+    <child link="gopigo3_body"/>
+    <parent link="base_link"/>
+  </joint>
+ <!--
+  <joint type="fixed" name="base_to_lidar">
+    <origin xyz="0.03 0 0.1126" rpy=" 0 0 0"/>
+    <parent link="base_link"/>
+    <child link="lidar"/>
+  </joint>
+ -->
 </robot>
